Commit message: clean up towed version

File: urdf/wheelie_bot.urdf (robot description, URDF)
Before this commit: robot Wheelie Bot, 6 links, 5 joints
Links:
- added link implement_base_platform, mass 1; collision box size=0.5 0.5 0.1; visual box size=0.5 1 0.1
- added link implement_base_platform_left_wheel, mass 1; collision cylinder length=0.1 radius=0.25; visual cylinder length=0.1 radius=0.25
- added link implement_base_platform_right_wheel, mass 1; collision cylinder length=0.1 radius=0.25; visual cylinder length=0.1 radius=0.25
- added link implement_connector, mass 0.5; collision box size=1 1 0.2; visual box size=2 0.1 0.1
- link base_link: mass 10 -> 25
- link front_caster_wheel: mass 5 -> 0.5; geometry collision cylinder length=0.1 radius=0.065; visual cylinder length=0.1 radius=0.065
Joints:
- added joint implement_base_platform_left_wheel_joint: type continuous, parent implement_base_platform, child implement_base_platform_left_wheel, origin xyz=0 0.6 0 rpy=-1.57075 0 0, axis 0 0 1, limit effort=30 velocity=10.0
- added joint implement_base_platform_right_wheel_joint: type continuous, parent implement_base_platform, child implement_base_platform_right_wheel, origin xyz=0 -0.6 0 rpy=-1.57075 0 0, axis 0 0 -1, limit effort=30 velocity=10.0
- added joint implement_connector_base_platform_joint: type fixed, parent implement_connector, child implement_base_platform, origin xyz=-2 -0 -0.25 rpy=0 0 0
- added joint implement_connector_joint: type revolute, parent base_link, child implement_connector, origin xyz=-0.5 -0 0.25 rpy=0 0 0, axis 0 0 1, limit lower=-1.4 upper=1.4 effort=1000.0 velocity=0.5

Commit message: Changed IMU and GPS Transforms.

File: urdf/wheelie_bot.urdf (robot description, URDF)
Before this commit: robot Wheelie Bot, 10 links, 9 joints
Links:
- removed link base_bottom
- added link base_footprint
- added link gps_link, mass 0.00001; collision box size=0.1 0.1 0.1; visual box size=0.1 0.1 0.1
- added link imu_link, mass 0.00001; collision box size=0.1 0.1 0.1; visual box size=0.1 0.1 0.1
Joints:
- removed joint base_bottom_to_link
- added joint base_footprint_to_link: type fixed, parent base_footprint, child base_link, origin xyz=0 0 0.25
- added joint gps_base_link_tf: type fixed, parent base_link, child gps_link, origin xyz=0 0 0.75
- added joint imu_base_link_tf: type fixed, parent base_link, child imu_link, origin xyz=0 0 0.20

Commit message: Included a laser scan in the urdf description

File: urdf/wheelie_bot.urdf (robot description, URDF)
Before this commit: robot Wheelie Bot, 12 links, 11 joints
Links:
- added link hokuyo_link, mass 0.00001; collision box size=0.01 0.01 0.01; visual mesh filename=package://wheelie_bot/meshes/hokuyo.dae
Joints:
- added joint laser_base_link_tf: type fixed, parent base_link, child hokuyo_link, origin xyz=0.4 0 0.45
